File: mixer/mixer.kicad_sch (KiCad schematic)
At the start: 36 parts, among them J1 Conn_02x05_Odd_Even, J2 CV_IN1, J3 CV_OUT1, J4 CV_IN2, J5 CV_OUT2, J6 CV_IN3, J7 CV_OUT3, J8 MIX_OUT, SW1 SW_SPST, SW2 SW_SPST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

Commit message: sdsds
Parts:
- removed FB1, FB2: FerriteBead_Small, Inductor_SMD:L_0805_2012Metric_Pad1.05x1.20mm_HandSolder, symbol Device:FerriteBead_Small
- removed SW1, SW2, SW3: SW_SPST, benjiaomodular:ToggleSwitch_MTS-101_SPST, symbol Switch:SW_SPST
- removed U2, U3, U4, U5: 100k, mong:PTL45, symbol _mong:Pot_led
- added R11, R12, R13: 22k, Resistor_SMD:R_0805_2012Metric_Pad1.20x1.40mm_HandSolder, symbol Device:R_US
- added RV1, RV2, RV3, RV4: 100k, Potentiometer_THT:Potentiometer_Bourns_PTA3043_Single_Slide, symbol Device:R_Potentiometer_US
- added SW1, SW2, SW3, SW4: SW_SPDT, benjiaomodular:ToggleSwitch_MTS-102_SPDT, symbol Switch:SW_SPDT
- J1: footprint Connector_IDC:IDC-Header_2x05_P2.54mm_Vertical -> Connector_PinHeader_2.54mm:PinHeader_2x05_P2.54mm_Vertical
- J2: value CV_IN1 -> Jack
- J3: value CV_OUT1 -> Jack
- J4: value CV_IN2 -> Jack
- J5: value CV_OUT2 -> Jack
- J6: value CV_IN3 -> Jack
- J7: value CV_OUT3 -> Jack
- J8: value MIX_OUT -> Jack
- R1, R2, R3: value 100k -> 1k
- R10, R8, R9: value 10k -> 100k
- U1: footprint Package_DIP:DIP-8_W7.62mm -> Package_SO:SOIC-8_3.9x4.9mm_P1.27mm
Connections:
- net +12V: now also R11.2, R12.2, R13.2
- net GND: now also RV1.3, RV2.3, RV3.3, RV4.3, SW1.3 (C), SW2.3 (C), SW3.3 (C), SW4.3 (C); no longer R10.1, R8.1, R9.1
- net at R5.2, U1.1: now also SW4.1 (A); no longer R4.1
- net at R5.1, U1.2 (-): now also R10.2, R8.2, R9.2
- net at R3.1: now also RV3.2
- net at J4.2: now also R12.1
- net at J4.3: now also SW2.1 (A)
- net at J6.3: now also SW3.1 (A)
- net at D1.2 (A): now also J1.10 (Pin_10), J1.9 (Pin_9)
- net at R1.1: now also RV1.2
- net at D2.1 (K): now also J1.1 (Pin_1), J1.2 (Pin_2)
- net at R2.1: now also RV2.2
- net at J6.2: now also R13.1
- net at J2.2: now also R11.1
- net at J2.3: now also SW1.1 (A)
- new net: R4.1, RV4.2
- new net: RV2.1, SW2.2 (B)
- new net: J7.2, R10.1
- new net: RV4.1, SW4.2 (B)
- new net: RV1.1, SW1.2 (B)
- new net: J3.2, R8.1
- new net: RV3.1, SW3.2 (B)
- new net: J5.2, R9.1
- no-connect marks 3 -> 0
Other:
- note removed: "Bourns PTL45"
- moved on the sheet: C1, C2, C3, C4, J1, J2, J4, J6, J8, R1, R2, R3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

Commit message: fgdfg
Parts:
- J2, J3, J4, J5, J6, J7, J8: footprint THONK_PJ398SM-12 -> mong:Thonkiconn_J398SM_Vertical_CircularHoles
- RV1, RV2, RV3, RV4: footprint Potentiometer_THT:Potentiometer_Bourns_PTA3043_Single_Slide -> mong:Potentiometer_Bourns_PTA3043_Single_Slide
Changed lines of the file:
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@@
 			)
 		)
-		(property "Footprint" "Potentiometer_THT:Potentiometer_Bourns_PTA3043_Single_Slide"
+		(property "Footprint" "mong:Potentiometer_Bourns_PTA3043_Single_Slide"
 			(at 95.25 74.93 0)
 			(effects
@@
 			)
 		)
-		(property "Footprint" "THONK_PJ398SM-12"
+		(property "Footprint" "mong:Thonkiconn_J398SM_Vertical_CircularHoles"
 			(at 121.92 86.36 0)
 			(effects
@@
 			)
 		)
-		(property "Footprint" "THONK_PJ398SM-12"
+		(property "Footprint" "mong:Thonkiconn_J398SM_Vertical_CircularHoles"
 			(at 62.23 77.47 0)
 			(effects
@@
 			)
 		)
-		(property "Footprint" "Potentiometer_THT:Potentiometer_Bourns_PTA3043_Single_Slide"
+		(property "Footprint" "mong:Potentiometer_Bourns_PTA3043_Single_Slide"
 			(at 196.85 106.68 0)
 			(effects
@@
 			)
 		)
-		(property "Footprint" "THONK_PJ398SM-12"
+		(property "Footprint" "mong:Thonkiconn_J398SM_Vertical_CircularHoles"
 			(at 262.89 97.79 0)
 			(effects
@@
 			)
 		)
-		(property "Footprint" "Potentiometer_THT:Potentiometer_Bourns_PTA3043_Single_Slide"
+		(property "Footprint" "mong:Potentiometer_Bourns_PTA3043_Single_Slide"
 			(at 95.25 45.72 0)
 			(effects
@@
 			)
 		)
-		(property "Footprint" "THONK_PJ398SM-12"
+		(property "Footprint" "mong:Thonkiconn_J398SM_Vertical_CircularHoles"
 			(at 62.23 106.68 0)
 			(effects
@@
 			)
 		)
-		(property "Footprint" "THONK_PJ398SM-12"
+		(property "Footprint" "mong:Thonkiconn_J398SM_Vertical_CircularHoles"
 			(at 121.92 27.94 0)
 			(effects
@@
 			)
 		)
-		(property "Footprint" "Potentiometer_THT:Potentiometer_Bourns_PTA3043_Single_Slide"
+		(property "Footprint" "mong:Potentiometer_Bourns_PTA3043_Single_Slide"
 			(at 95.25 104.14 0)
 			(effects
@@
 			)
 		)
-		(property "Footprint" "THONK_PJ398SM-12"
+		(property "Footprint" "mong:Thonkiconn_J398SM_Vertical_CircularHoles"
 			(at 60.96 48.26 0)
 			(effects
@@
 			)
 		)
-		(property "Footprint" "THONK_PJ398SM-12"
+		(property "Footprint" "mong:Thonkiconn_J398SM_Vertical_CircularHoles"
 			(at 121.92 55.88 0)
 			(effects
