File: mixer/mixer.kicad_pcb (KiCad board)
At the start: 2 copper layers, 49 x 100 mm, 36 parts, among them J1 Conn_02x05_Odd_Even, J2 CV_IN1, J3 CV_OUT1, J4 CV_IN2, J5 CV_OUT2, J6 CV_IN3, J7 CV_OUT3, J8 MIX_OUT, SW1 SW_SPST, SW2 SW_SPST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

Commit message: sdsds
Parts:
- removed FB1, FB2: FerriteBead_Small, Inductor_SMD:L_0805_2012Metric_Pad1.05x1.20mm_HandSolder
- removed U2, U3, U4, U5: 100k, mong:PTL45
- added R11: 22k, Resistor_SMD:R_0805_2012Metric_Pad1.20x1.40mm_HandSolder, B.Cu at (206.0, 71.0)
- added R12: 22k, Resistor_SMD:R_0805_2012Metric_Pad1.20x1.40mm_HandSolder, B.Cu at (218.0, 71.5)
- added R13: 22k, Resistor_SMD:R_0805_2012Metric_Pad1.20x1.40mm_HandSolder, B.Cu at (229.5, 71.5)
- added RV1: 100k, Potentiometer_THT:Potentiometer_Bourns_PTA3043_Single_Slide, F.Cu at (207.7, 85.3)
- added RV2: 100k, Potentiometer_THT:Potentiometer_Bourns_PTA3043_Single_Slide, F.Cu at (219.5, 85.3)
- added RV3: 100k, Potentiometer_THT:Potentiometer_Bourns_PTA3043_Single_Slide, F.Cu at (231.2, 85.3)
- added RV4: 100k, Potentiometer_THT:Potentiometer_Bourns_PTA3043_Single_Slide, F.Cu at (239.8, 129.0)
- added SW4: SW_SPDT, benjiaomodular:ToggleSwitch_MTS-102_SPDT, F.Cu at (241.3, 139.8)
- J1: footprint Connector_IDC:IDC-Header_2x05_P2.54mm_Vertical -> Connector_PinHeader_2.54mm:PinHeader_2x05_P2.54mm_Vertical
- J2: value CV_IN1 -> Jack
- J3: value CV_OUT1 -> Jack
- J4: value CV_IN2 -> Jack
- J5: value CV_OUT2 -> Jack
- J6: value CV_IN3 -> Jack
- J7: value CV_OUT3 -> Jack
- J8: value MIX_OUT -> Jack
- R1, R2, R3: value 100k -> 1k
- R10, R8, R9: value 10k -> 100k; moved to B.Cu
- SW1, SW2, SW3: value SW_SPST -> SW_SPDT; footprint benjiaomodular:ToggleSwitch_MTS-101_SPST -> benjiaomodular:ToggleSwitch_MTS-102_SPDT
- U1: footprint Package_DIP:DIP-8_W7.62mm -> Package_SO:SOIC-8_3.9x4.9mm_P1.27mm
- moved R8 78.1 mm to (212.5, 64.5), turned to 0 degrees
- moved J1 78.0 mm to (247.0, 68.0), turned to 180 degrees
- moved C4 76.1 mm to (241.0, 71.5), turned to 90 degrees
- moved D2 74.6 mm to (240.5, 68.0), turned to 180 degrees
- moved R10 69.9 mm to (226.5, 67.0), turned to -90 degrees
- moved R9 58.6 mm to (223.0, 67.0), turned to -90 degrees
- moved C2 51.6 mm to (236.0, 70.5), turned to 90 degrees
- moved R2 50.3 mm to (212.5, 57.5), turned to 90 degrees
- moved R1 49.9 mm to (202.5, 57.5), turned to 90 degrees
- moved C3 47.3 mm to (241.0, 76.0), turned to -90 degrees
- moved R7 45.5 mm to (238.0, 57.0), turned to 90 degrees
- moved R3 45.0 mm to (225.5, 57.5), turned to 90 degrees
- moved C1 35.6 mm to (236.0, 78.5), turned to 90 degrees
- moved U1 32.9 mm to (229.5, 104.5), turned to 0 degrees
- moved D1 27.0 mm to (241.0, 81.0), turned to 0 degrees
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Connections:
- J1 pad 1: Net-(J1-Pin_1) -> Net-(D2-K)
- J1 pad 10: Net-(J1-Pin_10) -> Net-(D1-A)
- J1 pad 2: Net-(J1-Pin_1) -> Net-(D2-K)
- J1 pad 9: Net-(J1-Pin_10) -> Net-(D1-A)
- J2 pad 2: unconnected-(J2-Pad2) -> Net-(J2-Pad2)
- J4 pad 2: unconnected-(J4-Pad2) -> Net-(J4-Pad2)
- J5 pad 2: Net-(J3-Pad2) -> Net-(J5-Pad2)
- J6 pad 2: unconnected-(J6-Pad2) -> Net-(J6-Pad2)
- J7 pad 2: Net-(J3-Pad2) -> Net-(J7-Pad2)
- R10 pad 1: GND -> Net-(J7-Pad2)
- R10 pad 2: Net-(R10-Pad2) -> Net-(U1A--)
- R5 pad 2: Net-(R4-Pad1) -> Net-(SW4-A)
- R8 pad 1: GND -> Net-(J3-Pad2)
- R8 pad 2: Net-(R8-Pad2) -> Net-(U1A--)
- R9 pad 1: GND -> Net-(J5-Pad2)
- R9 pad 2: Net-(R9-Pad2) -> Net-(U1A--)
- U1 pad 1: Net-(R4-Pad1) -> Net-(SW4-A)
Routing:
- net Net-(SW3-A): track 0.00 -> 59.7 mm
- net Net-(SW2-A): track 0.00 -> 59.7 mm
- net Net-(SW1-A): track 0.00 -> 59.7 mm
- net Net-(R6-Pad2): track 0.00 -> 57.8 mm, vias 0 -> 2
- net Net-(SW2-B): track 0.00 -> 56.8 mm
- net Net-(SW1-B): track 0.00 -> 56.8 mm
- net Net-(SW3-B): track 0.00 -> 56.2 mm
- net Net-(U1A--): track 0.00 -> 56.0 mm, vias 0 -> 2
- net -12V: track 0.00 -> 44.9 mm, vias 0 -> 2
- net Net-(SW4-A): track 0.00 -> 38.9 mm, vias 0 -> 1
- net Net-(R4-Pad1): track 0.00 -> 33.7 mm
- net Net-(R2-Pad1): track 0.00 -> 28.3 mm, vias 0 -> 2
- net Net-(R3-Pad1): track 0.00 -> 28.1 mm, vias 0 -> 1
- net Net-(R1-Pad1): track 0.00 -> 27.5 mm
- net +12V: track 0.00 -> 23.0 mm, vias 0 -> 5
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
Commit message: sdasd
Parts:
- J2, J3, J4, J5, J6, J7, J8: footprint Seattle_Synths:THONK_PJ398SM-12 -> mong:Thonkiconn_J398SM_Vertical_CircularHoles
- RV1, RV2, RV3, RV4: footprint Potentiometer_THT:Potentiometer_Bourns_PTA3043_Single_Slide -> mong:Potentiometer_Bourns_PTA3043_Single_Slide
- moved J3 6.78 mm to (206.2, 64.3), turned to 180 degrees
- moved J5 6.78 mm to (217.9, 64.3), turned to 180 degrees
- moved J7 6.78 mm to (229.7, 64.3), turned to 180 degrees
- moved J8 6.78 mm to (241.5, 64.3), turned to 180 degrees
- moved J2 6.28 mm to (206.2, 64.2), turned to 0 degrees
- moved J4 6.28 mm to (217.9, 64.2), turned to 0 degrees
- moved J6 6.28 mm to (229.7, 64.2), turned to 0 degrees
- moved RV1 0.22 mm to (207.9, 85.2)
- moved RV2 0.22 mm to (219.7, 85.2)
- moved RV3 0.22 mm to (231.4, 85.2)
- moved RV4 0.22 mm to (239.9, 128.9)
Routing:
- net Net-(U1A--): track 56.0 -> 58.6 mm
- net Net-(SW3-B): track 56.2 -> 57.3 mm
Other:
- board text added: "so naughty"
- board text added: "supercalm meeks v1.0"
